File: gu10-12v-lamp.kicad_pcb (KiCad board)
At the start: 2 copper layers, 50 x 50 mm, 25 parts

Commit message: Add: Gerber files
Parts:
- removed C1: DNP, Capacitor_SMD:C_0805_2012Metric
Routing:
- net Net-(D3-Pad1): track 8.24 -> 0.00 mm
- net Net-(D11-Pad1): track 8.01 -> 0.00 mm
- net Net-(D10-Pad2): track 7.31 -> 0.00 mm
- net Net-(D5-Pad1): track 7.11 -> 0.00 mm
- net Net-(D4-Pad1): track 6.90 -> 0.00 mm
- net Net-(D2-Pad1): track 6.82 -> 0.00 mm
- net Net-(D6-Pad1): track 6.80 -> 0.00 mm
- net Net-(D12-Pad1): track 6.62 -> 0.00 mm
- net Net-(D4-Pad2): track 3.58 -> 0.00 mm
- net Net-(D11-Pad2): track 3.90 -> 0.34 mm
- net Net-(D3-Pad2): track 3.44 -> 0.00 mm
- net Net-(D2-Pad2): track 3.43 -> 0.00 mm
- net Net-(D1-Pad4): track 6.38 -> 5.48 mm
- net GND: vias 88 -> 78
- added copper zone on F.Cu, net Net-(D10-Pad2)
- added copper zone on F.Cu, net Net-(D11-Pad1)
- added copper zone on F.Cu, net Net-(D11-Pad2)
- added copper zone on F.Cu, net Net-(D12-Pad1)
- added copper zone on F.Cu, net Net-(D2-Pad1)
- added copper zone on F.Cu, net Net-(D2-Pad2)
- added copper zone on F.Cu, net Net-(D3-Pad1)
- added copper zone on F.Cu, net Net-(D3-Pad2)
- added copper zone on F.Cu, net Net-(D4-Pad1)
- added copper zone on F.Cu, net Net-(D4-Pad2)
- added copper zone on F.Cu, net Net-(D5-Pad1)
- added copper zone on F.Cu, net Net-(D6-Pad1)
Other:
- board text added: "ISS B"

Commit message: Add: Issue B assets
Parts:
- D10, D11, D12, D13, D2, D3, D4, D5, D6, D7, D8, D9: footprint LED_SMD:LED_PLCC_2835_Custom -> 2835-led.kicad_mod:LED_PLCC_2835
- R1, R2, R3, R4: value 20R -> 39R
Other:
- board text added: "2.5mm NPTH x 4"
- board text added: "Between GU10 Pins (3.2mm PTH x 2)"
- board text added: "Between Mounting Holes"
- board text added: "Board Radius"
- board text added: "Radius of 4 Mounting Holes"
