File: gu10-12v-lamp.sch (KiCad schematic (older format))
At the start: 23 parts

Commit message: Add: Issue B assets
Parts:
- D1: Vendor (none) -> Digi-Key; Vendor 10of GBP (none) -> 0.41; Vendor SKU (none) -> DF01SA-E3/77GICT-ND
- D10, D11, D12, D13, D2, D3, D4, D5, D6, D7, D8, D9: footprint LED_SMD:LED_PLCC_2835_Custom -> 2835-led.kicad_mod:LED_PLCC_2835; Vendor (none) -> Digi-Key; Vendor 10of GBP (none) -> 0.01500; Vendor SKU (none) -> 2138-JB2835AWT-W-U30GA0000-N0000001CT-ND
- R1, R2, R3, R4: value 20R -> 39R; Vendor (none) -> Digi-Key; Vendor 10of GBP (none) -> 0.181; Vendor SKU (none) -> RMCF2512JT39R0CT-ND
Changed lines of the file:
@@
 Title "GU10 12V Lamp"
 Date ""
-Rev "ISS A"
+Rev "ISS B"
 Comp "damow.net"
 Comment1 ""
@@
 F 2 "Diode_SMD:Diode_Bridge_Vishay_DFS" H 3650 3500 50  0001 C CNN
 F 3 "~" H 3650 3500 50  0001 C CNN
+F 4 "Digi-Key" H 3650 3500 50  0001 C CNN "Vendor"
+F 5 "0.41" H 3650 3500 50  0001 C CNN "Vendor 10of GBP"
+F 6 "DF01SA-E3/77GICT-ND" H 3650 3500 50  0001 C CNN "Vendor SKU"
 	1    3650 3500
 	1    0    0    -1
@@
 P 6200 3150
 F 0 "R2" V 5993 3150 50  0000 C CNN
-F 1 "20R" V 6084 3150 50  0000 C CNN
+F 1 "39R" V 6084 3150 50  0000 C CNN
 F 2 "Resistor_SMD:R_2512_6332Metric" V 6130 3150 50  0001 C CNN
 F 3 "~" H 6200 3150 50  0001 C CNN
+F 4 "Digi-Key" H 6200 3150 50  0001 C CNN "Vendor"
+F 5 "0.181" H 6200 3150 50  0001 C CNN "Vendor 10of GBP"
+F 6 "RMCF2512JT39R0CT-ND" H 6200 3150 50  0001 C CNN "Vendor SKU"
 	1    6200 3150
 	0    1    1    0
@@
 P 6200 2050
 F 0 "R1" V 5993 2050 50  0000 C CNN
-F 1 "20R" V 6084 2050 50  0000 C CNN
+F 1 "39R" V 6084 2050 50  0000 C CNN
 F 2 "Resistor_SMD:R_2512_6332Metric" V 6130 2050 50  0001 C CNN
 F 3 "~" H 6200 2050 50  0001 C CNN
+F 4 "Digi-Key" H 6200 2050 50  0001 C CNN "Vendor"
+F 5 "0.181" H 6200 2050 50  0001 C CNN "Vendor 10of GBP"
+F 6 "RMCF2512JT39R0CT-ND" H 6200 2050 50  0001 C CNN "Vendor SKU"
 	1    6200 2050
 	0    1    1    0
@@
 F 0 "D9" H 8093 2895 50  0000 C CNN
 F 1 "LED" H 8093 2986 50  0000 C CNN
-F 2 "LED_SMD:LED_PLCC_2835_Custom" H 8100 3150 50  0001 C CNN
+F 2 "2835-led.kicad_mod:LED_PLCC_2835" H 8100 3150 50  0001 C CNN
 F 3 "~" H 8100 3150 50  0001 C CNN
+F 4 "Digi-Key" H 8100 3150 50  0001 C CNN "Vendor"
+F 5 "" H 8100 3150 50  0001 C CNN "Vendor 10of"
+F 6 "2138-JB2835AWT-W-U30GA0000-N0000001CT-ND" H 8100 3150 50  0001 C CNN "Vendor SKU"
+F 7 "0.01500" H 8100 3150 50  0001 C CNN "Vendor 10of GBP"
 	1    8100 3150
 	-1   0    0    1
@@
 F 0 "D6" H 7443 2895 50  0000 C CNN
 F 1 "LED" H 7443 2986 50  0000 C CNN
-F 2 "LED_SMD:LED_PLCC_2835_Custom" H 7450 3150 50  0001 C CNN
+F 2 "2835-led.kicad_mod:LED_PLCC_2835" H 7450 3150 50  0001 C CNN
 F 3 "~" H 7450 3150 50  0001 C CNN
+F 4 "Digi-Key" H 7450 3150 50  0001 C CNN "Vendor"
+F 5 "" H 7450 3150 50  0001 C CNN "Vendor 10of"
+F 6 "2138-JB2835AWT-W-U30GA0000-N0000001CT-ND" H 7450 3150 50  0001 C CNN "Vendor SKU"
+F 7 "0.01500" H 7450 3150 50  0001 C CNN "Vendor 10of GBP"
 	1    7450 3150
 	-1   0    0    1
@@
 F 0 "D3" H 6793 2895 50  0000 C CNN
 F 1 "LED" H 6793 2986 50  0000 C CNN
-F 2 "LED_SMD:LED_PLCC_2835_Custom" H 6800 3150 50  0001 C CNN
+F 2 "2835-led.kicad_mod:LED_PLCC_2835" H 6800 3150 50  0001 C CNN
 F 3 "~" H 6800 3150 50  0001 C CNN
+F 4 "Digi-Key" H 6800 3150 50  0001 C CNN "Vendor"
+F 5 "0.01500" H 6800 3150 50  0001 C CNN "Vendor 10of GBP"
+F 6 "2138-JB2835AWT-W-U30GA0000-N0000001CT-ND" H 6800 3150 50  0001 C CNN "Vendor SKU"
 	1    6800 3150
 	-1   0    0    1
@@
 F 0 "D8" H 8093 1795 50  0000 C CNN
 F 1 "LED" H 8093 1886 50  0000 C CNN
-F 2 "LED_SMD:LED_PLCC_2835_Custom" H 8100 2050 50  0001 C CNN
+F 2 "2835-led.kicad_mod:LED_PLCC_2835" H 8100 2050 50  0001 C CNN
 F 3 "~" H 8100 2050 50  0001 C CNN
+F 4 "Digi-Key" H 8100 2050 50  0001 C CNN "Vendor"
+F 5 "" H 8100 2050 50  0001 C CNN "Vendor 10of"
+F 6 "2138-JB2835AWT-W-U30GA0000-N0000001CT-ND" H 8100 2050 50  0001 C CNN "Vendor SKU"
+F 7 "0.01500" H 8100 2050 50  0001 C CNN "Vendor 10of GBP"
 	1    8100 2050
 	-1   0    0    1
@@
 F 0 "D5" H 7443 1795 50  0000 C CNN
 F 1 "LED" H 7443 1886 50  0000 C CNN
-F 2 "LED_SMD:LED_PLCC_2835_Custom" H 7450 2050 50  0001 C CNN
+F 2 "2835-led.kicad_mod:LED_PLCC_2835" H 7450 2050 50  0001 C CNN
 F 3 "~" H 7450 2050 50  0001 C CNN
+F 4 "Digi-Key" H 7450 2050 50  0001 C CNN "Vendor"
+F 5 "" H 7450 2050 50  0001 C CNN "Vendor 10of"
+F 6 "2138-JB2835AWT-W-U30GA0000-N0000001CT-ND" H 7450 2050 50  0001 C CNN "Vendor SKU"
+F 7 "0.01500" H 7450 2050 50  0001 C CNN "Vendor 10of GBP"
 	1    7450 2050
 	-1   0    0    1
@@
 F 0 "D2" H 6793 1795 50  0000 C CNN
 F 1 "LED" H 6793 1886 50  0000 C CNN
-F 2 "LED_SMD:LED_PLCC_2835_Custom" H 6800 2050 50  0001 C CNN
+F 2 "2835-led.kicad_mod:LED_PLCC_2835" H 6800 2050 50  0001 C CNN
 F 3 "~" H 6800 2050 50  0001 C CNN
+F 4 "Digi-Key" H 6800 2050 50  0001 C CNN "Vendor"
+F 5 "" H 6800 2050 50  0001 C CNN "Vendor 10of"
+F 6 "2138-JB2835AWT-W-U30GA0000-N0000001CT-ND" H 6800 2050 50  0001 C CNN "Vendor SKU"
+F 7 "0.01500" H 6800 2050 50  0001 C CNN "Vendor 10of GBP"
 	1    6800 2050
 	-1   0    0    1
@@
 P 6200 4300
 F 0 "R3" V 5993 4300 50  0000 C CNN
-F 1 "20R" V 6084 4300 50  0000 C CNN
+F 1 "39R" V 6084 4300 50  0000 C CNN
 F 2 "Resistor_SMD:R_2512_6332Metric" V 6130 4300 50  0001 C CNN
 F 3 "~" H 6200 4300 50  0001 C CNN
+F 4 "Digi-Key" H 6200 4300 50  0001 C CNN "Vendor"
+F 5 "0.181" H 6200 4300 50  0001 C CNN "Vendor 10of GBP"
+F 6 "RMCF2512JT39R0CT-ND" H 6200 4300 50  0001 C CNN "Vendor SKU"
 	1    6200 4300
 	0    1    1    0
@@
 F 0 "D10" H 8093 4045 50  0000 C CNN
 F 1 "LED" H 8093 4136 50  0000 C CNN
-F 2 "LED_SMD:LED_PLCC_2835_Custom" H 8100 4300 50  0001 C CNN
+F 2 "2835-led.kicad_mod:LED_PLCC_2835" H 8100 4300 50  0001 C CNN
 F 3 "~" H 8100 4300 50  0001 C CNN
+F 4 "Digi-Key" H 8100 4300 50  0001 C CNN "Vendor"
+F 5 "" H 8100 4300 50  0001 C CNN "Vendor 10of"
+F 6 "2138-JB2835AWT-W-U30GA0000-N0000001CT-ND" H 8100 4300 50  0001 C CNN "Vendor SKU"
+F 7 "0.01500" H 8100 4300 50  0001 C CNN "Vendor 10of GBP"
 	1    8100 4300
 	-1   0    0    1
@@
 F 0 "D7" H 7443 4045 50  0000 C CNN
 F 1 "LED" H 7443 4136 50  0000 C CNN
-F 2 "LED_SMD:LED_PLCC_2835_Custom" H 7450 4300 50  0001 C CNN
+F 2 "2835-led.kicad_mod:LED_PLCC_2835" H 7450 4300 50  0001 C CNN
 F 3 "~" H 7450 4300 50  0001 C CNN
+F 4 "Digi-Key" H 7450 4300 50  0001 C CNN "Vendor"
+F 5 "" H 7450 4300 50  0001 C CNN "Vendor 10of"
+F 6 "2138-JB2835AWT-W-U30GA0000-N0000001CT-ND" H 7450 4300 50  0001 C CNN "Vendor SKU"
+F 7 "0.01500" H 7450 4300 50  0001 C CNN "Vendor 10of GBP"
 	1    7450 4300
 	-1   0    0    1
@@
 F 0 "D4" H 6793 4045 50  0000 C CNN
 F 1 "LED" H 6793 4136 50  0000 C CNN
-F 2 "LED_SMD:LED_PLCC_2835_Custom" H 6800 4300 50  0001 C CNN
+F 2 "2835-led.kicad_mod:LED_PLCC_2835" H 6800 4300 50  0001 C CNN
 F 3 "~" H 6800 4300 50  0001 C CNN
+F 4 "Digi-Key" H 6800 4300 50  0001 C CNN "Vendor"
+F 5 "" H 6800 4300 50  0001 C CNN "Vendor 10of"
+F 6 "2138-JB2835AWT-W-U30GA0000-N0000001CT-ND" H 6800 4300 50  0001 C CNN "Vendor SKU"
+F 7 "0.01500" H 6800 4300 50  0001 C CNN "Vendor 10of GBP"
 	1    6800 4300
 	-1   0    0    1
@@
 P 6200 5500
 F 0 "R4" V 5993 5500 50  0000 C CNN
-F 1 "20R" V 6084 5500 50  0000 C CNN
+F 1 "39R" V 6084 5500 50  0000 C CNN
 F 2 "Resistor_SMD:R_2512_6332Metric" V 6130 5500 50  0001 C CNN
 F 3 "~" H 6200 5500 50  0001 C CNN
+F 4 "Digi-Key" H 6200 5500 50  0001 C CNN "Vendor"
+F 5 "0.181" H 6200 5500 50  0001 C CNN "Vendor 10of GBP"
+F 6 "RMCF2512JT39R0CT-ND" H 6200 5500 50  0001 C CNN "Vendor SKU"
 	1    6200 5500
 	0    1    1    0
@@
 F 0 "D13" H 8093 5245 50  0000 C CNN
 F 1 "LED" H 8093 5336 50  0000 C CNN
-F 2 "LED_SMD:LED_PLCC_2835_Custom" H 8100 5500 50  0001 C CNN
+F 2 "2835-led.kicad_mod:LED_PLCC_2835" H 8100 5500 50  0001 C CNN
 F 3 "~" H 8100 5500 50  0001 C CNN
+F 4 "Digi-Key" H 8100 5500 50  0001 C CNN "Vendor"
+F 5 "" H 8100 5500 50  0001 C CNN "Vendor 10of"
+F 6 "2138-JB2835AWT-W-U30GA0000-N0000001CT-ND" H 8100 5500 50  0001 C CNN "Vendor SKU"
+F 7 "0.01500" H 8100 5500 50  0001 C CNN "Vendor 10of GBP"
 	1    8100 5500
 	-1   0    0    1
@@
 F 0 "D12" H 7443 5245 50  0000 C CNN
 F 1 "LED" H 7443 5336 50  0000 C CNN
-F 2 "LED_SMD:LED_PLCC_2835_Custom" H 7450 5500 50  0001 C CNN
+F 2 "2835-led.kicad_mod:LED_PLCC_2835" H 7450 5500 50  0001 C CNN
 F 3 "~" H 7450 5500 50  0001 C CNN
+F 4 "Digi-Key" H 7450 5500 50  0001 C CNN "Vendor"
+F 5 "" H 7450 5500 50  0001 C CNN "Vendor 10of"
+F 6 "2138-JB2835AWT-W-U30GA0000-N0000001CT-ND" H 7450 5500 50  0001 C CNN "Vendor SKU"
+F 7 "0.01500" H 7450 5500 50  0001 C CNN "Vendor 10of GBP"
 	1    7450 5500
 	-1   0    0    1
@@
 F 0 "D11" H 6793 5245 50  0000 C CNN
 F 1 "LED" H 6793 5336 50  0000 C CNN
-F 2 "LED_SMD:LED_PLCC_2835_Custom" H 6800 5500 50  0001 C CNN
+F 2 "2835-led.kicad_mod:LED_PLCC_2835" H 6800 5500 50  0001 C CNN
 F 3 "~" H 6800 5500 50  0001 C CNN
+F 4 "Digi-Key" H 6800 5500 50  0001 C CNN "Vendor"
+F 5 "" H 6800 5500 50  0001 C CNN "Vendor 10of"
+F 6 "2138-JB2835AWT-W-U30GA0000-N0000001CT-ND" H 6800 5500 50  0001 C CNN "Vendor SKU"
+F 7 "0.01500" H 6800 5500 50  0001 C CNN "Vendor 10of GBP"
 	1    6800 5500
 	-1   0    0    1
